Commit message: Se actualiza el urdf y se importan los primeros modelos del brazo robotico(base del robot, base rotacional y link1

File: urdf/mi_brazo.urdf (robot description, URDF)
Before this commit: robot Mi_Brazo, 6 links, 5 joints
Links:
- removed link end_effector
- removed link link2
- removed link link3
- removed link link4
- added link base_rotation, mass 3; collision mesh filename=urdf/mesh/Base_Rotacional.stl scale=0.001 0.001 0.001; visual mesh filename=urdf/mesh/Base_Rotacional.stl scale=0.001 0.001 0.001
- link base_link: geometry collision mesh filename=urdf/mesh/Base_Brazo_Robotico.stl scale=0.001 0.001 0.001; visual mesh filename=urdf/mesh/Base_Brazo_Robotico.stl scale=0.001 0.001 0.001
- link link1: geometry collision mesh filename=urdf/mesh/Link1.stl scale=0.001 0.001 0.001; visual mesh filename=urdf/mesh/Link1.stl scale=0.001 0.001 0.001
Joints:
- removed joint elbow_joint
- removed joint wrist_pitch_joint
- removed joint wrist_roll_joint
- joint base_joint: child link1 -> base_rotation; limit lower=-3.1416 upper=3.1416 effort=200 velocity=5 -> lower=-3.1416 upper=3.1416 effort=300 velocity=5; origin xyz=0 0 0.05 rpy=0 0 0 -> xyz=0 0 0.08 rpy=0 0 0
- joint shoulder_joint: axis 1 0 0 -> 0 1 0; child link2 -> link1; limit lower=-1.57 upper=1.57 effort=100 velocity=3 -> lower=-1.57 upper=1.57 effort=200 velocity=3; origin xyz=0 0 0.5 rpy=0 0 0 -> xyz=0 0 0.045 rpy=0 0 0; parent link1 -> base_rotation

Commit message: Se carga el link2 y se ajustan detalles en cuanto a los origenes de los componentes para que las juntas coincidan en la simulacion :D

File: urdf/mi_brazo.urdf (robot description, URDF)
Before this commit: robot Mi_Brazo, 3 links, 2 joints
Links:
- added link link2, mass 1; collision mesh filename=urdf/mesh/Link2.stl scale=0.001 0.001 0.001; visual mesh filename=urdf/mesh/Link2.stl scale=0.001 0.001 0.001
Joints:
- added joint elbow_joint: type revolute, parent link1, child link2, origin xyz=0.504 0 0 rpy=0 0 0, axis 0 1 0, limit lower=-1.57 upper=1.57 effort=150 velocity=3

Commit message: Se importan los componentes principales del brazo robotico y se carga en pybullet para revisar en simulacion

File: urdf/mi_brazo.urdf (robot description, URDF)
Before this commit: robot Mi_Brazo, 4 links, 3 joints
Links:
- added link Link3, mass 1; collision mesh filename=urdf/mesh/Link3.stl scale=0.001 0.001 0.001; visual mesh filename=urdf/mesh/Link3.stl scale=0.001 0.001 0.001
- added link Link4, mass 1; collision mesh filename=urdf/mesh/Link4.stl scale=0.001 0.001 0.001; visual mesh filename=urdf/mesh/Link4.stl scale=0.001 0.001 0.001
Joints:
- added joint wrist_pitch_joint: type revolute, parent link2, child Link3, origin xyz=0.424 0 0 rpy=0 0 0, axis 0 1 0, limit lower=-1.57 upper=1.57 effort=100 velocity=3
- added joint wrist_yaw_joint: type revolute, parent Link3, child Link4, origin xyz=0.345 0 0 rpy=0 0 0, axis 0 1 0, limit lower=-1.57 upper=1.57 effort=100 velocity=3

Commit message: Se crean jerarquias y modulos de cada RL de momento dos partes y  se crea simulacion de brazo individual para comprobar coordenadas del brazo

File: urdf/mi_brazo.urdf (robot description, URDF)
Before this commit: robot Mi_Brazo, 6 links, 5 joints
Links:
- added link end_effector, mass 0.0001
- link Link3: mass 1 -> 0.1; geometry collision mesh filename=urdf/mesh/Link3.stl scale=0.00035 0.00035 0.00035; visual mesh filename=urdf/mesh/Link3.stl scale=0.00035 0.00035 0.00035
- link Link4: mass 1 -> 0.08; geometry collision mesh filename=urdf/mesh/Link4.stl scale=0.00035 0.00035 0.00035; visual mesh filename=urdf/mesh/Link4.stl scale=0.00035 0.00035 0.00035
- link base_link: mass 10 -> 1.5; geometry collision mesh filename=urdf/mesh/Base_Brazo_Robotico.stl scale=0.00035 0.00035 0.00035; visual mesh filename=urdf/mesh/Base_Brazo_Robotico.stl scale=0.00035 0.00035 0.00035
- link base_rotation: mass 3 -> 0.4; geometry collision mesh filename=urdf/mesh/Base_Rotacional.stl scale=0.00035 0.00035 0.00035; visual mesh filename=urdf/mesh/Base_Rotacional.stl scale=0.00035 0.00035 0.00035
- link link1: mass 2 -> 0.3; geometry collision mesh filename=urdf/mesh/Link1.stl scale=0.00035 0.00035 0.00035; visual mesh filename=urdf/mesh/Link1.stl scale=0.00035 0.00035 0.00035
- link link2: mass 1 -> 0.2; geometry collision mesh filename=urdf/mesh/Link2.stl scale=0.00035 0.00035 0.00035; visual mesh filename=urdf/mesh/Link2.stl scale=0.00035 0.00035 0.00035
Joints:
- added joint end_effector_joint: type fixed, parent Link4, child end_effector, origin xyz=0.0525 0 0
- joint base_joint: limit lower=-3.1416 upper=3.1416 effort=300 velocity=5 -> lower=-3.14 upper=3.14 effort=300 velocity=5; origin xyz=0 0 0.08 rpy=0 0 0 -> xyz=0 0 0.028
- joint elbow_joint: limit lower=-1.57 upper=1.57 effort=150 velocity=3 -> lower=-3.14 upper=3.14 effort=300 velocity=3; origin xyz=0.504 0 0 rpy=0 0 0 -> xyz=0.1764 0 0
- joint shoulder_joint: limit lower=-1.57 upper=1.57 effort=200 velocity=3 -> lower=-3.14 upper=3.14 effort=300 velocity=3; origin xyz=0 0 0.045 rpy=0 0 0 -> xyz=0 0 0.0157
- joint wrist_pitch_joint: limit lower=-1.57 upper=1.57 effort=100 velocity=3 -> lower=-3.14 upper=3.14 effort=100 velocity=3; origin xyz=0.424 0 0 rpy=0 0 0 -> xyz=0.1484 0 0
- joint wrist_yaw_joint: limit lower=-1.57 upper=1.57 effort=100 velocity=3 -> lower=-3.14 upper=3.14 effort=100 velocity=3; origin xyz=0.345 0 0 rpy=0 0 0 -> xyz=0.1207 0 0
